File: pcb/reflex-io-board/reflex-io-board.sch (KiCad schematic (older format))
At the start: 111 parts, among them J1 RJ45, J10 Barrel_Jack_MountingPin, J11 Barrel_Jack_MountingPin, J12 Conn_02x04_Odd_Even, J2 RJ45, J3 RJ45, J4 RJ45, J5 USB_B, J6 Conn_02x05_Odd_Even, J7 Barrel_Jack_MountingPin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

Commit message: Order in
Connections:
- net labels added: GNDD
- wire segments 624 -> 625
Changed lines of the file:
@@
 EESchema Schematic File Version 4
+LIBS:reflex-io-board-cache
 EELAYER 30 0
 EELAYER END
@@
 Connection ~ 3900 5150
 $Comp
-L Interface_UART:SP3485EN U8
-U 1 1 5FCA13F1
-P 4750 7100
-F 0 "U8" H 4850 6700 50  0000 C CNN
-F 1 "SP3485EN" H 4450 6700 50  0000 C CNN
-F 2 "Package_SO:SOIC-8_3.9x4.9mm_P1.27mm" H 5800 6750 50  0001 C CIN
-F 3 "http://www.icbase.com/pdf/SPX/SPX00480106.pdf" H 4750 7100 50  0001 C CNN
-	1    4750 7100
-	1    0    0    -1
-$EndComp
-$Comp
 L Device:R R34
 U 1 1 5FCA13F7
@@
 Wire Wire Line
 	8250 6500 8950 6500
-Wire Wire Line
-	8950 6500 8950 6950
 Connection ~ 8250 6500
 Wire Wire Line
@@
 Wire Wire Line
 	6950 9750 6800 9750
-$Comp
-L power:GND #PWR039
-U 1 1 60151260
-P 6800 9500
-F 0 "#PWR039" H 6800 9250 50  0001 C CNN
-F 1 "GND" H 6805 9327 50  0000 C CNN
-F 2 "" H 6800 9500 50  0001 C CNN
-F 3 "" H 6800 9500 50  0001 C CNN
-	1    6800 9500
-	-1   0    0    1
-$EndComp
-Wire Wire Line
-	6800 9500 6800 9550
 Connection ~ 6800 9550
 Wire Wire Line
@@
 Text GLabel 1450 10150 2    50   Input ~ 0
 USART3_TX-
-Text GLabel 1450 10350 2    50   Input ~ 0
-USART3_CK+
 Text GLabel 1450 10250 2    50   Input ~ 0
+USART3_CK+
+Text GLabel 1450 10350 2    50   Input ~ 0
 USART3_CK-
 $Comp
@@
 	5300 10000 5300 9900
 Connection ~ 5050 10000
+$Comp
+L power:GNDD #PWR0101
+U 1 1 5F6D34EF
+P 6800 9800
+F 0 "#PWR0101" H 6800 9550 50  0001 C CNN
+F 1 "GNDD" H 6950 9800 50  0000 C CNN
+F 2 "" H 6800 9800 50  0001 C CNN
+F 3 "" H 6800 9800 50  0001 C CNN
+	1    6800 9800
+	1    0    0    -1
+$EndComp
+Wire Wire Line
+	6800 9800 6800 9750
+Connection ~ 6800 9750
+$Comp
+L power:PWR_FLAG #FLG0103
+U 1 1 5F72EE4C
+P 7250 9450
+F 0 "#FLG0103" H 7250 9525 50  0001 C CNN
+F 1 "PWR_FLAG" H 7250 9623 50  0000 C CNN
+F 2 "" H 7250 9450 50  0001 C CNN
+F 3 "~" H 7250 9450 50  0001 C CNN
+	1    7250 9450
+	1    0    0    -1
+$EndComp
+Wire Wire Line
+	7250 9550 7250 9450
+Connection ~ 7250 9550
+Wire Wire Line
+	8950 6500 8950 6950
+$Comp
+L Interface_UART:SP3485EN U8
+U 1 1 5FCA13F1
+P 4750 7100
+F 0 "U8" H 4850 6700 50  0000 C CNN
+F 1 "SP3485EN" H 4450 6700 50  0000 C CNN
+F 2 "Package_SO:SOIC-8_3.9x4.9mm_P1.27mm" H 5800 6750 50  0001 C CIN
+F 3 "http://www.icbase.com/pdf/SPX/SPX00480106.pdf" H 4750 7100 50  0001 C CNN
+	1    4750 7100
+	1    0    0    -1
+$EndComp
 $EndSCHEMATC
