File: io-board.kicad_pcb (KiCad board)
At the start: 4 copper layers, 270 x 34 mm, 112 parts, among them J1 RJ45, J10 Barrel_Jack_MountingPin, J11 Barrel_Jack_MountingPin, J12 Conn_02x04_Odd_Even, J2 RJ45, J3 RJ45, J4 RJ45, J5 USB_B, J6 Conn_02x05_Odd_Even, J7 Barrel_Jack_MountingPin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

Commit message: Safe margins for no standoffs
Parts:
- moved J10 18.5 mm to (73.5, 125.5)
- moved J9 16.5 mm to (61.5, 125.5)
- moved J11 14.5 mm to (85.5, 120.5)
- moved J7 12.8 mm to (61.5, 120.5), turned to 180 degrees
- moved J8 10.7 mm to (73.5, 120.5), turned to 180 degrees
- moved G*** 7.50 mm to (39.2, 112.8)
- moved C1 7.00 mm to (110.8, 114.2)
- moved C10 7.00 mm to (95.2, 113.8)
- moved C11 7.00 mm to (149.4, 114.4)
- moved C12 7.00 mm to (173.0, 114.5)
- moved C13 7.00 mm to (121.0, 114.2)
- moved C14 7.00 mm to (227.5, 126.5)
- moved C15 7.00 mm to (205.8, 114.0)
- moved C16 7.00 mm to (197.5, 114.2)
- moved C17 7.00 mm to (225.0, 138.0)
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Other:
- outline, holes or cut-outs redrawn

Commit message: RS-485 transceiver fixes - production
Parts:
- removed C10, C11, C12, C13: 0.1u, Capacitor_SMD:C_0603_1608Metric
- removed G***: LOGO, local:reflex-dance-logo-28
- removed R44, R47, R50: 120R, Resistor_SMD:R_0603_1608Metric
- removed R45, R46, R48, R49, R51: 360R, Resistor_SMD:R_0603_1608Metric
- removed U10, U11, U12, U9: SP3485EN, Package_SO:SOIC-8_3.9x4.9mm_P1.27mm
- R1, R17, R18, R19, R2, R20, R3, R36, R37, R38, R39, R4: value 0R -> 10k
- R12, R15, R25, R28, R31, R34, R6, R9: value 120R -> 100R
- R40, R42, R43: value 360R -> 10k
- R41: value 120R -> 10k
- moved R42 80.2 mm to (180.8, 111.0)
- moved R41 66.9 mm to (165.1, 108.2), turned to 180 degrees
- moved R43 17.9 mm to (136.4, 108.2), turned to 180 degrees
- moved R40 17.0 mm to (110.7, 108.2), turned to 180 degrees
- moved R19 15.1 mm to (195.8, 111.3)
- moved R18 7.90 mm to (165.1, 111.0), turned to -90 degrees
- moved R20 7.90 mm to (136.7, 111.0), turned to -90 degrees
- moved R37 7.86 mm to (157.2, 110.5)
- moved R39 7.82 mm to (128.8, 110.2), turned to -90 degrees
- moved R17 7.74 mm to (110.7, 111.0), turned to -90 degrees
- moved R1 7.36 mm to (118.1, 111.0)
- moved R2 7.25 mm to (172.2, 110.5)
- moved R36 6.86 mm to (102.1, 110.2)
- moved R38 6.08 mm to (179.1, 111.0), turned to -90 degrees
- moved R4 5.93 mm to (141.7, 108.2), turned to 0 degrees
Connections:
- J1 pad 4: USART1_CK- -> unconnected-(J1-Pad4)
- J1 pad 5: USART1_CK+ -> unconnected-(J1-Pad5)
- J2 pad 4: USART3_CK- -> unconnected-(J2-Pad4)
- J2 pad 5: USART3_CK+ -> unconnected-(J2-Pad5)
- J3 pad 4: USART2_CK0- -> unconnected-(J3-Pad4)
- J3 pad 5: USART2_CK0+ -> unconnected-(J3-Pad5)
- J4 pad 4: USART2_CK1- -> unconnected-(J4-Pad4)
- J4 pad 5: USART2_CK1+ -> unconnected-(J4-Pad5)
- J6 pad 10: Net-(J6-Pad10) -> unconnected-(J6-Pad10)
- J6 pad 3: Net-(J6-Pad3) -> unconnected-(J6-Pad3)
- J6 pad 9: Net-(J6-Pad9) -> unconnected-(J6-Pad9)
- R1 pad 1: USART1_RX -> USART1_RX_DR
- R1 pad 2: Net-(R1-Pad2) -> GND
- R17 pad 1: USART1_TX -> Net-(R17-Pad1)
- R17 pad 2: Net-(R17-Pad2) -> GND
- R18 pad 1: USART2_TX0 -> Net-(R18-Pad1)
- R18 pad 2: Net-(R18-Pad2) -> GND
- R19 pad 1: USART2_TX1 -> Net-(R19-Pad1)
- R19 pad 2: Net-(R19-Pad2) -> GND
- R2 pad 1: USART2_RX0 -> USART2_RX0_DR
- R2 pad 2: Net-(R2-Pad2) -> GND
- R20 pad 1: USART3_TX -> Net-(R20-Pad1)
- R20 pad 2: Net-(R20-Pad2) -> GND
- R3 pad 1: USART2_RX1 -> USART2_RX1_DR
- R3 pad 2: Net-(R3-Pad2) -> GND
- R36 pad 1: USART1_CK -> USART1_TX_DR
- R36 pad 2: Net-(R36-Pad2) -> GND
- R37 pad 1: USART2_CK0 -> USART2_TX0_DR
- R37 pad 2: Net-(R37-Pad2) -> GND
- R38 pad 1: USART2_CK1 -> USART2_TX1_DR
- R38 pad 2: Net-(R38-Pad2) -> GND
- R39 pad 1: USART3_CK -> USART3_TX_DR
- R39 pad 2: Net-(R39-Pad2) -> GND
- R4 pad 1: USART3_RX -> USART3_RX_DR
- R4 pad 2: Net-(R4-Pad2) -> GND
- R40 pad 2: USART1_CK+ -> Net-(R40-Pad2)
- R41 pad 1: USART1_CK+ -> +3V3
- R41 pad 2: USART1_CK- -> Net-(R41-Pad2)
- R42 pad 1: USART1_CK- -> +3V3
- R42 pad 2: GND -> Net-(R42-Pad2)
- R43 pad 2: USART2_CK0+ -> Net-(R43-Pad2)
- U1 pad 2: GND -> USART1_RX_DR
- U1 pad 4: Net-(R1-Pad2) -> Net-(R17-Pad1)
- U14 pad 14: USART2_CK0 -> unconnected-(U14-Pad14)
- U14 pad 20: USART3_CK_DR -> unconnected-(U14-Pad20)
- U14 pad 25: USART3_CK -> unconnected-(U14-Pad25)
- U14 pad 26: USART1_CK_DR -> unconnected-(U14-Pad26)
- U14 pad 29: USART1_CK -> unconnected-(U14-Pad29)
- U14 pad 41: USART2_CK1 -> unconnected-(U14-Pad41)
- U14 pad 43: USART2_CK1_DR -> unconnected-(U14-Pad43)
- U14 pad 46: USART2_CK0_DR -> unconnected-(U14-Pad46)
- U2 pad 2: GND -> USART2_RX0_DR
- U2 pad 4: Net-(R2-Pad2) -> Net-(R18-Pad1)
- U3 pad 2: GND -> USART2_RX1_DR
- U3 pad 4: Net-(R3-Pad2) -> Net-(R19-Pad1)
- U4 pad 2: GND -> USART3_RX_DR
- U4 pad 4: Net-(R4-Pad2) -> Net-(R20-Pad1)
- U5 pad 1: Net-(R17-Pad2) -> Net-(R40-Pad2)
- U5 pad 2: GND -> USART1_TX_DR
- U6 pad 1: Net-(R18-Pad2) -> Net-(R41-Pad2)
- U6 pad 2: GND -> USART2_TX0_DR
- U7 pad 1: Net-(R19-Pad2) -> Net-(R42-Pad2)
- U7 pad 2: GND -> USART2_TX1_DR
- U8 pad 1: Net-(R20-Pad2) -> Net-(R43-Pad2)
- U8 pad 2: GND -> USART3_TX_DR
Routing:
- net USART1_CK_DR: track 176.7 -> 0.00 mm, vias 2 -> 0
- net USART1_CK: track 166.7 -> 0.00 mm, vias 6 -> 0
- net GND: track 320.1 -> 194.1 mm, vias 23 -> 29
- net USART3_CK: track 117.3 -> 0.00 mm, vias 4 -> 0
- net USART3_CK_DR: track 106.1 -> 0.00 mm, vias 2 -> 0
- net USART2_CK0: track 73.1 -> 0.00 mm, vias 2 -> 0
- net USART2_CK0_DR: track 65.0 -> 0.00 mm
- net +3V3: track 242.4 -> 184.8 mm, vias 17 -> 16
- net USART2_CK1: track 53.0 -> 0.00 mm, vias 2 -> 0
- net USART2_CK1_DR: track 47.8 -> 0.00 mm, vias 2 -> 0
- net USART2_CK1+: track 21.7 -> 0.00 mm
- net USART3_CK+: track 20.3 -> 0.00 mm
- net USART1_RX: track 146.0 -> 127.7 mm
- net USART1_CK+: track 18.2 -> 0.00 mm
- net USART2_CK0+: track 17.2 -> 0.00 mm
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Other:
- net class Default removed
